File: PlacaAlimentacion/PlacaAlimentacion/PlacaAlimentacion.sch (KiCad schematic (older format))
At the start: 17 parts, among them J1 Conn_01x03_Male, J2 Screw_Terminal_01x04, U1 LM741, U2 LM741, U3 LM741

Commit message: Comienzo de diseño Placa Alimentacion
Parts:
- removed CA1: CP470u, Capacitor_THT:CP_Radial_D10.0mm_P5.00mm, symbol Device:CP
- removed CC1: CP100u, Capacitor_THT:CP_Radial_D8.0mm_P3.80mm, symbol Device:CP
- removed J1: Conn_01x03_Male, Connector_PinHeader_2.54mm:PinHeader_1x03_P2.54mm_Horizontal, symbol Connector:Conn_01x03_Male
- removed JM1, JM2: Screw_Terminal_01x02, TerminalBlock_Phoenix:TerminalBlock_Phoenix_MKDS-1,5-2-5.08_1x02_P5.08mm_Horizontal, symbol Connector:Screw_Terminal_01x02
- added C1: CAP104, Capacitor_THT:CP_Radial_D6.3mm_P2.50mm, symbol pspice:CAP
- added C2, C5: CP47u, Capacitor_THT:CP_Radial_D6.3mm_P2.50mm, symbol Device:CP
- added C3, C4: CP10u, Capacitor_THT:CP_Radial_D6.3mm_P2.50mm, symbol Device:CP
- added D1, D2, D3, D4: LED, LED_THT:LED_D5.0mm, symbol Device:LED
- added D5, D5231: D_Zener, Diode_THT:D_DO-35_SOD27_P10.16mm_Horizontal, symbol Device:D_Zener
- added F1, F2: Fuse, FusibleAmericano:R_Axial_DIN0411_L9.9mm_D3.6mm_P20.32mm_Horizontal, symbol Device:Fuse
- added J1, J5: Conn_01x04_Male, Connector_PinHeader_2.54mm:PinHeader_1x04_P2.54mm_Horizontal, symbol Connector:Conn_01x04_Male
- added J3, J4: USB_A, Connector_USB:USB_A_Wuerth_61400826021_Horizontal_Stacked, symbol Connector:USB_A
- added J6, J7, J8: Screw_Terminal_01x04, TerminalBlock_Phoenix:TerminalBlock_Phoenix_MKDS-1,5-4-5.08_1x04_P5.08mm_Horizontal, symbol Connector:Screw_Terminal_01x04
- added R10, R11, R12, R120, R1k1, R1k2, R360, R9: R, Resistor_THT:R_Axial_DIN0207_L6.3mm_D2.5mm_P7.62mm_Horizontal, symbol Device:R
- added SW1: SW_DPST, SwitchPower:SW_CuK_JS202011AQN_DPDT_Angled, symbol Switch:SW_DPST
- added U4: LM1084-ADJ, Package_TO_SOT_THT:TO-220-3_Vertical, symbol Regulator_Linear:LM1084-ADJ
- added U5: LM7805_TO220, Package_TO_SOT_THT:TO-220-3_Vertical, symbol Regulator_Linear:LM7805_TO220
Connections:
- net BAT1: now also C3.1, C4.1, SW1.4, U4.3 (VI), U5.1 (VI)
- net BAT2: now also J6.4 (Pin_4), J7.4 (Pin_4), R10.1, R9.1, SW1.2
- net VBATT1: now also D5.1 (K), J1.4 (Pin_4), R1k1.1; no longer U1.3 (+), U1.6
- net VBATT2: now also D5231.1 (K), J1.2 (Pin_2), R1k2.1; no longer R8.1, U3.6
- net +24V renamed GND2
- net GND2: now also F1.2, J8.1 (Pin_1)
- net +5V renamed GND1
- net GND1: now also R3.2, R4.2, R7.2, U1.4 (V-), U2.4 (V-), U3.4 (V-), C1.2, C4.2, C5.2, D1.1 (K), D2.1 (K), D3.1 (K), D4.1 (K), D5.2 (A), D5231.2 (A), J5.1 (Pin_1), J5.3 (Pin_3), J6.2 (Pin_2), J7.2 (Pin_2), U5.2 (GND)
- removed net GND: J2.2 (Pin_2), R3.2, R4.2, R7.2, U1.4 (V-), U2.4 (V-), U3.4 (V-)
- net GNDPWR: no longer names the net of J2.3 (Pin_3)
- new net: R1k1.2, U1.3 (+), U1.6
- new net: R1k2.2, R8.1, U3.6
- new net: F2.1, SW1.1
- new net: F1.1, SW1.3
- new net: D1.2 (A), R9.2
- new net: R120.2, R360.1, U4.1 (ADJ)
- new net: D2.2 (A), R10.2
- new net: D3.2 (A), R11.2
- new net: D4.2 (A), R12.2
- new net NC: J1.1 (Pin_1), J1.3 (Pin_3)
- new net PWR_GND: J6.3 (Pin_3), J7.3 (Pin_3)
- new net RPI_GND: C2.2, C3.2, J3.4 (GND), J4.4 (GND), R360.2
- new net RPI_VDD: C2.1, J3.1 (VBUS), J4.1 (VBUS), R12.1, R120.1, U4.2 (VO)
- new net VDD: C1.1, C5.1, J5.2 (Pin_2), J5.4 (Pin_4), J6.1 (Pin_1), J7.1 (Pin_1), R11.1, U5.3 (VO)
- new net VOLBAT2: F2.2, J8.4 (Pin_4)
Other:
- note added: "Alimentacion1\n"
- note added: "Alimentacion2\n"
- note added: "Bateria1"
- note added: "Bateria2"
- note added: "Master SW\n"
- note added: "Visualizacion\n"
- note removed: "Alimentación"
- note removed: "Salida Motores\n"
- moved on the sheet: J2, R1, R2, R3, R4, R5, R6, R7, R8, U1, U2, U3
